Commit message: move_group node now runs everything, fixed small warning in the depth camera urdf and the  collision meshes are being loaded now, rviz still not working

File: ros2_ws/src/spraying_pathways/urdf/depth_camera.urdf.xacro (robot description, xacro)
@@ -12,5 +12,7 @@
       <visual>
         <geometry><box size="0.05 0.05 0.05"/></geometry>
-        <material name="Gray"/>
+        <material name="Gray">
+          <color rgba="0.5 0.5 0.5 1.0"/>
+        </material>
       </visual>
       <collision>
