Commit message: mock execution works in rviz

File: ros2_ws/src/spraying_pathways/urdf/my_robot.urdf.xacro (robot description, xacro)
@@ -22,3 +22,39 @@
   <xacro:depth_camera_ee parent_link="$(arg tf_prefix)wrist_3_link" sim_gazebo="$(arg sim_gazebo)" />
   <!-- <xacro:lidar_sensor parent_link="$(arg tf_prefix)tool0" tf_prefix="$(arg tf_prefix)" sim_gazebo="$(arg sim_gazebo)" /> -->
+  <ros2_control name="MockSystem" type="system">
+    <hardware>
+      <plugin>mock_components/GenericSystem</plugin>
+      <param name="calculate_dynamics">true</param>
+    </hardware>
+    <joint name="$(arg tf_prefix)shoulder_pan_joint">
+      <command_interface name="position"/>
+      <state_interface name="position"><param name="initial_value">0.0</param></state_interface>
+      <state_interface name="velocity"/>
+    </joint>
+    <joint name="$(arg tf_prefix)shoulder_lift_joint">
+      <command_interface name="position"/>
+      <state_interface name="position"><param name="initial_value">-1.5708</param></state_interface>
+      <state_interface name="velocity"/>
+    </joint>
+    <joint name="$(arg tf_prefix)elbow_joint">
+      <command_interface name="position"/>
+      <state_interface name="position"><param name="initial_value">0.0</param></state_interface>
+      <state_interface name="velocity"/>
+    </joint>
+    <joint name="$(arg tf_prefix)wrist_1_joint">
+      <command_interface name="position"/>
+      <state_interface name="position"><param name="initial_value">-1.5708</param></state_interface>
+      <state_interface name="velocity"/>
+    </joint>
+    <joint name="$(arg tf_prefix)wrist_2_joint">
+      <command_interface name="position"/>
+      <state_interface name="position"><param name="initial_value">0.0</param></state_interface>
+      <state_interface name="velocity"/>
+    </joint>
+    <joint name="$(arg tf_prefix)wrist_3_joint">
+      <command_interface name="position"/>
+      <state_interface name="position"><param name="initial_value">0.0</param></state_interface>
+      <state_interface name="velocity"/>
+    </joint>
+  </ros2_control>
 </robot>

Commit message: gz_ros2_control now build from source inside control, explicit ros2 control tags in urdf, gazebo render engine  change in launch file because of black screen in vm

File: ros2_ws/src/spraying_pathways/urdf/my_robot.urdf.xacro (robot description, xacro)
@@ -19,38 +19,37 @@
   <!-- <xacro:include filename="$(find spraying_pathways)/urdf/2d_lidar.urdf.xacro" /> -->
   <!-- Custom sensors -->
-  <xacro:depth_camera parent_link="$(arg tf_prefix)base_link" sim_gazebo="$(arg sim_gazebo)" />
-  <xacro:depth_camera_ee parent_link="$(arg tf_prefix)wrist_3_link" sim_gazebo="$(arg sim_gazebo)" />
-  <!-- <xacro:lidar_sensor parent_link="$(arg tf_prefix)tool0" tf_prefix="$(arg tf_prefix)" sim_gazebo="$(arg sim_gazebo)" /> -->
-  <ros2_control name="MockSystem" type="system">
+  <xacro:depth_camera parent_link="$(arg prefix)base_link" sim_gazebo="$(arg sim_gazebo)" />
+  <xacro:depth_camera_ee parent_link="$(arg prefix)wrist_3_link" sim_gazebo="$(arg sim_gazebo)" />
+  <!-- <xacro:lidar_sensor parent_link="$(arg prefix)tool0" tf_prefix="$(arg prefix)" sim_gazebo="$(arg sim_gazebo)" /> -->
+  <ros2_control name="GazeboSimSystem" type="system">
     <hardware>
-      <plugin>mock_components/GenericSystem</plugin>
-      <param name="calculate_dynamics">true</param>
+      <plugin>gz_ros2_control/GazeboSimSystem</plugin>
     </hardware>
-    <joint name="$(arg tf_prefix)shoulder_pan_joint">
+    <joint name="$(arg prefix)shoulder_pan_joint">
       <command_interface name="position"/>
       <state_interface name="position"><param name="initial_value">0.0</param></state_interface>
       <state_interface name="velocity"/>
     </joint>
-    <joint name="$(arg tf_prefix)shoulder_lift_joint">
+    <joint name="$(arg prefix)shoulder_lift_joint">
       <command_interface name="position"/>
       <state_interface name="position"><param name="initial_value">-1.5708</param></state_interface>
       <state_interface name="velocity"/>
     </joint>
-    <joint name="$(arg tf_prefix)elbow_joint">
+    <joint name="$(arg prefix)elbow_joint">
       <command_interface name="position"/>
       <state_interface name="position"><param name="initial_value">0.0</param></state_interface>
       <state_interface name="velocity"/>
     </joint>
-    <joint name="$(arg tf_prefix)wrist_1_joint">
+    <joint name="$(arg prefix)wrist_1_joint">
       <command_interface name="position"/>
       <state_interface name="position"><param name="initial_value">-1.5708</param></state_interface>
       <state_interface name="velocity"/>
     </joint>
-    <joint name="$(arg tf_prefix)wrist_2_joint">
+    <joint name="$(arg prefix)wrist_2_joint">
       <command_interface name="position"/>
       <state_interface name="position"><param name="initial_value">0.0</param></state_interface>
       <state_interface name="velocity"/>
     </joint>
-    <joint name="$(arg tf_prefix)wrist_3_joint">
+    <joint name="$(arg prefix)wrist_3_joint">
       <command_interface name="position"/>
       <state_interface name="position"><param name="initial_value">0.0</param></state_interface>
@@ -58,3 +57,8 @@
     </joint>
   </ros2_control>
+  <gazebo>
+    <plugin filename="libgz_ros2_control-system.so" name="gz_ros2_control::GazeboSimROS2ControlPlugin">
+      <parameters>$(arg simulation_controllers)</parameters>
+    </plugin>
+  </gazebo>
 </robot>
