Commit message: added camera collision box to suppress warning, modified main launch to file to include obstacle_tracking and epoxy_visualizer. Started working on obstacle ovoidance

File: ros2_ws/src/spraying_pathways/urdf/depth_camera_ee.urdf.xacro (robot description, xacro)
@@ -13,4 +13,10 @@
         </material>
         </visual>
+        <collision>
+        <origin xyz="0 0 0" rpy="0 0 0"/>
+        <geometry>
+            <box size="0.02 0.02 0.02"/>
+        </geometry>
+        </collision>
     </link>
     <joint name="wrist_3-camera_joint" type="fixed">
